File: RedPill_board/RedPill_board.kicad_sch (KiCad schematic)
At the start: 62 parts, among them J3 Conn_01x26, J4 Conn_01x26, U1 STM32F103CBTx, U2 AMS1117-3.3, Y1 8MHz

Commit message: Sent to fab.
Parts:
- removed Y1: 8MHz, Crystal:Crystal_SMD_3225-4Pin_3.2x2.5mm, symbol Device:Crystal_GND24
- added Y1: 8MHz, Crystal:Crystal_SMD_5032-2Pin_5.0x3.2mm, symbol Device:Crystal
- C?: value 2u2 -> 4.7uF
Connections:
- net PGM_OSC_IN: now also Y1.1
- net PGM_OSC_OUT: now also Y1.2
Changed lines of the file:
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@@
     (stroke (width 0) (type default))
   )
-  (wire (pts (xy 51.435 60.96) (xy 59.69 60.96))
-    (stroke (width 0) (type default))
-  )
   (wire (pts (xy 127 67.31) (xy 132.08 67.31))
     (stroke (width 0) (type default))
@@
     (stroke (width 0) (type default))
   )
+  (wire (pts (xy 52.07 60.96) (xy 59.69 60.96))
+    (stroke (width 0) (type default))
+  )
   (wire (pts (xy 52.07 182.88) (xy 52.07 181.61))
     (stroke (width 0) (type default))
@@
     (stroke (width 0) (type default))
   )
-  (wire (pts (xy 38.735 60.96) (xy 43.815 60.96))
-    (stroke (width 0) (type default))
-  )
   (wire (pts (xy 227.33 31.115) (xy 227.33 33.02))
     (stroke (width 0) (type default))
@@
     (stroke (width 0) (type default))
   )
+  (wire (pts (xy 38.735 60.96) (xy 44.45 60.96))
+    (stroke (width 0) (type default))
+  )
   (wire (pts (xy 114.3 173.99) (xy 120.65 173.99))
     (stroke (width 0) (type default))
@@
     )
   )
+  (symbol (lib_id "Device:Crystal") (at 48.26 60.96 0) (unit 1)
+    (in_bom yes) (on_board yes) (dnp no) (fields_autoplaced)
+    (property "Reference" "Y1" (at 48.26 54.61 0)
+      (effects (font (size 1.27 1.27)))
+    )
+    (property "Value" "8MHz" (at 48.26 57.15 0)
+      (effects (font (size 1.27 1.27)))
+    )
+    (property "Footprint" "Crystal:Crystal_SMD_5032-2Pin_5.0x3.2mm" (at 48.26 60.96 0)
+      (effects (font (size 1.27 1.27)) hide)
+    )
+    (property "Datasheet" "~" (at 48.26 60.96 0)
+      (effects (font (size 1.27 1.27)) hide)
+    )
+    (pin "1")
+    (pin "2")
+    (instances
+      (project "RedPill_board"
+        (path "/2aa92989-679b-41e6-b5fc-2a171f9ac1b8"
+          (reference "Y1") (unit 1)
+        )
+      )
+    )
+  )
   (symbol (lib_id "MCU_ST_STM32F4:STM32F401RCTx") (at 228.6 97.79 0) (unit 1)
     (in_bom yes) (on_board yes) (dnp no) (fields_autoplaced)
@@
     )
   )
-  (symbol (lib_id "power:GND") (at 47.625 55.88 180) (unit 1)
-    (in_bom yes) (on_board yes) (dnp no) (fields_autoplaced)
-    (property "Reference" "#PWR?" (at 47.625 49.53 0)
-      (effects (font (size 1.27 1.27)) hide)
-    )
-    (property "Value" "GND" (at 47.625 52.07 0)
-      (effects (font (size 1.27 1.27)))
-    )
-    (property "Footprint" "" (at 47.625 55.88 0)
-      (effects (font (size 1.27 1.27)) hide)
-    )
-    (property "Datasheet" "" (at 47.625 55.88 0)
-      (effects (font (size 1.27 1.27)) hide)
-    )
-    (pin "1")
-    (instances
-      (project "stlinkes_devboard"
-        (path "/11450504-0e54-4d07-ac36-3601830b54ed"
-          (reference "#PWR?") (unit 1)
-        )
-      )
-      (project "RedPill_board"
-        (path "/2aa92989-679b-41e6-b5fc-2a171f9ac1b8"
-          (reference "#PWR046") (unit 1)
-        )
-      )
-    )
-  )
   (symbol (lib_id "power:GND") (at 140.97 142.875 0) (unit 1)
     (in_bom yes) (on_board yes) (dnp no) (fields_autoplaced)
@@
       (effects (font (size 1.27 1.27)) (justify left))
     )
-    (property "Value" "2u2" (at 207.645 135.89 0)
+    (property "Value" "4.7uF" (at 207.645 135.89 0)
       (effects (font (size 1.27 1.27)) (justify left))
     )
@@
     )
   )
-  (symbol (lib_id "power:GND") (at 47.625 66.04 0) (unit 1)
-    (in_bom yes) (on_board yes) (dnp no) (fields_autoplaced)
-    (property "Reference" "#PWR?" (at 47.625 72.39 0)
-      (effects (font (size 1.27 1.27)) hide)
-    )
-    (property "Value" "GND" (at 47.625 70.485 0)
-      (effects (font (size 1.27 1.27)))
-    )
-    (property "Footprint" "" (at 47.625 66.04 0)
-      (effects (font (size 1.27 1.27)) hide)
-    )
-    (property "Datasheet" "" (at 47.625 66.04 0)
-      (effects (font (size 1.27 1.27)) hide)
-    )
-    (pin "1")
-    (instances
-      (project "stlinkes_devboard"
-        (path "/11450504-0e54-4d07-ac36-3601830b54ed"
-          (reference "#PWR?") (unit 1)
-        )
-      )
-      (project "RedPill_board"
-        (path "/2aa92989-679b-41e6-b5fc-2a171f9ac1b8"
-          (reference "#PWR041") (unit 1)
-        )
-      )
-    )
-  )
   (symbol (lib_id "Device:R") (at 29.21 162.56 180) (unit 1)
     (in_bom yes) (on_board yes) (dnp no) (fields_autoplaced)
@@
         )
       )
-    )
-  )
-  (symbol (lib_id "Device:Crystal_GND24") (at 47.625 60.96 0) (unit 1)
-    (in_bom yes) (on_board yes) (dnp no)
-    (property "Reference" "Y1" (at 52.705 56.515 0)
-      (effects (font (size 1.27 1.27)))
-    )
-    (property "Value" "8MHz" (at 53.975 58.42 0)
-      (effects (font (size 1.27 1.27)))
-    )
-    (property "Footprint" "Crystal:Crystal_SMD_3225-4Pin_3.2x2.5mm" (at 47.625 60.96 0)
-      (effects (font (size 1.27 1.27)) hide)
-    )
-    (property "Datasheet" "~" (at 47.625 60.96 0)
-      (effects (font (size 1.27 1.27)) hide)
-    )
-    (pin "1")
-    (pin "2")
-    (pin "3")
-    (pin "4")
-    (instances
-      (project "RedPill_board"
-        (path "/2aa92989-679b-41e6-b5fc-2a171f9ac1b8"
-          (reference "Y1") (unit 1)
-        )
-      )
